File: pcb.kicad_pcb (KiCad board)
At the start: 2 copper layers, 65 x 56 mm, 50 parts, among them J1 Raspberry_Pi_2_3, J10 Conn_01x03_Male, J11 Conn_01x03_Male, J12 Conn_01x03_Male, J13 Conn_01x03_Male, J14 Conn_01x02_Male, J16 Conn_01x02_Male, J17 Conn_01x02_Male, J2 Conn_01x03_Male, J3 Conn_01x03_Male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

Commit message: final version sent to fabrication
Parts:
- added D1: LED, LED_SMD:LED_0603_1608Metric, F.Cu at (115.2, 80.9)
- added R10: 1k, Resistor_SMD:R_0603_1608Metric, F.Cu at (110.6, 80.9)
- moved C15 3.42 mm to (127.9, 92.7), turned to -90 degrees
- moved C5 2.41 mm to (142.4, 92.1)
- moved L1 1.31 mm to (150.5, 104.5)
- moved J1 0.82 mm to (101.3, 75.8)
- moved D5 0.76 mm to (146.7, 91.9)
- moved R2 0.51 mm to (134.5, 93.3)
- moved R3 0.51 mm to (134.5, 96.5)
- moved Q4 0.25 mm to (130.4, 96.0)
Routing:
- net LV_SCL: track 0.00 -> 18.6 mm, vias 0 -> 1
- net 5VPi: track 51.6 -> 35.0 mm, vias 3 -> 2
- net +5V: track 82.0 -> 93.8 mm, vias 0 -> 2
- net Net-(C5-Pad1): track 24.9 -> 30.6 mm
- net Net-(D1-Pad2): track 0.00 -> 3.02 mm
- net Net-(C5-Pad2): track 0.00 -> 2.87 mm
- net Net-(R2-Pad2): track 4.29 -> 3.78 mm
- net GNDD: vias 30 -> 32
Other:
- outline, holes or cut-outs redrawn
