File: pcb.kicad_sch (KiCad schematic)
At the start: 49 parts, among them J1 Raspberry_Pi_2_3, J10 Conn_01x03_Male, J11 Conn_01x03_Male, J12 Conn_01x03_Male, J13 Conn_01x03_Male, J14 Conn_01x02_Male, J16 Conn_01x02_Male, J17 Conn_01x02_Male, J2 Conn_01x03_Male, J3 Conn_01x03_Male, J4 Conn_01x02_Male, J5 Conn_01x02_Male, J6 Conn_01x03_Male, J7 Conn_01x03_Male, J8 Conn_01x03_Male, J9 Conn_01x03_Male, Q1 SI2306, Q2 Si2306, Q4 AO3407, U1 TPS54xxxDDA, U2 DMMT3906W-7-F, U3 PCA9685PW

Commit message: final version sent to fabrication
Parts:
- added D1: LED, LED_SMD:LED_0603_1608Metric, symbol Device:LED
- added R10: 1k, Resistor_SMD:R_0603_1608Metric, symbol Device:R
- Q1: value SI2306 -> BSS138A
- Q2: value Si2306 -> BSS138A
Connections:
- net 5VPi: now also R10.2
- net GNDD: now also D1.1 (K)
- new net: D1.2 (A), R10.1
Changed lines of the file:
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@@
   (junction (at 157.48 31.75) (diameter 0) (color 0 0 0 0)
   )
+  (junction (at 157.48 48.26) (diameter 0) (color 0 0 0 0)
+  )
   (junction (at 148.59 142.24) (diameter 0) (color 0 0 0 0)
   )
@@
   )
   (wire (pts (xy 162.56 30.48) (xy 162.56 31.75))
+    (stroke (width 0) (type default) (color 0 0 0 0))
+  )
+  (wire (pts (xy 157.48 48.26) (xy 157.48 50.8))
     (stroke (width 0) (type default) (color 0 0 0 0))
   )
@@
     (effects (font (size 1.27 1.27)) (justify left))
     (property "Intersheet References" "${INTERSHEET_REFS}" (id 0) (at 259.1666 105.3306 0)
+      (effects (font (size 1.27 1.27)) (justify left) hide)
+    )
+  )
+  (global_label "5VPi" (shape input) (at 34.29 172.72 90) (fields_autoplaced)
+    (effects (font (size 1.27 1.27)) (justify left))
+    (property "Intersheet References" "${INTERSHEET_REFS}" (id 0) (at 34.2106 166.2229 90)
       (effects (font (size 1.27 1.27)) (justify left) hide)
     )
@@
     (in_bom yes) (on_board yes)
     (property "Reference" "Q1" (id 0) (at 128.27 101.6 90))
-    (property "Value" "SI2306" (id 1) (at 128.27 104.14 90))
+    (property "Value" "BSS138A" (id 1) (at 128.27 104.14 90))
     (property "Footprint" "Package_TO_SOT_SMD:SOT-23" (id 2) (at 125.73 99.06 0)
       (effects (font (size 1.27 1.27)) hide)
     )
-    (property "Datasheet" "https://www.mouser.com/datasheet/2/427/si2306bd-1766202.pdf" (id 3) (at 128.27 93.98 0)
+    (property "Datasheet" "https://www.mouser.com/datasheet/2/258/BSS138A_SOT_23_-2510176.pdf" (id 3) (at 128.27 93.98 0)
       (effects (font (size 1.27 1.27)) hide)
     )
@@
     (pin "1")
   )
+  (symbol (lib_id "power:GNDD") (at 34.29 187.96 0) (unit 1)
+    (in_bom yes) (on_board yes)
+    (property "Reference" "#PWR025" (id 0) (at 34.29 194.31 0)
+      (effects (font (size 1.27 1.27)) hide)
+    )
+    (property "Value" "GNDD" (id 1) (at 34.29 191.135 0)
+      (effects (font (size 1.27 1.27)) hide)
+    )
+    (property "Footprint" "" (id 2) (at 34.29 187.96 0)
+      (effects (font (size 1.27 1.27)) hide)
+    )
+    (property "Datasheet" "" (id 3) (at 34.29 187.96 0)
+      (effects (font (size 1.27 1.27)) hide)
+    )
+    (pin "1")
+  )
   (symbol (lib_id "Connector:Conn_01x03_Male") (at 223.52 72.39 180) (unit 1)
     (in_bom yes) (on_board yes) (fields_autoplaced)
@@
     (in_bom yes) (on_board yes) (fields_autoplaced)
     (property "Reference" "Q2" (id 0) (at 128.27 123.19 90))
-    (property "Value" "Si2306" (id 1) (at 128.27 125.73 90))
+    (property "Value" "BSS138A" (id 1) (at 128.27 125.73 90))
     (property "Footprint" "Package_TO_SOT_SMD:SOT-23" (id 2) (at 125.73 120.65 0)
       (effects (font (size 1.27 1.27)) hide)
     )
-    (property "Datasheet" "https://www.mouser.com/datasheet/2/427/si2306bd-1766202.pdf" (id 3) (at 128.27 115.57 0)
+    (property "Datasheet" "https://www.mouser.com/datasheet/2/258/BSS138A_SOT_23_-2510176.pdf" (id 3) (at 128.27 115.57 0)
       (effects (font (size 1.27 1.27)) hide)
     )
@@
     (pin "2")
   )
+  (symbol (lib_id "Device:LED") (at 34.29 184.15 90) (unit 1)
+    (in_bom yes) (on_board yes) (fields_autoplaced)
+    (property "Reference" "D1" (id 0) (at 37.211 184.9028 90)
+      (effects (font (size 1.27 1.27)) (justify right))
+    )
+    (property "Value" "LED" (id 1) (at 37.211 187.4397 90)
+      (effects (font (size 1.27 1.27)) (justify right))
+    )
+    (property "Footprint" "LED_SMD:LED_0603_1608Metric" (id 2) (at 34.29 184.15 0)
+      (effects (font (size 1.27 1.27)) hide)
+    )
+    (property "Datasheet" "~" (id 3) (at 34.29 184.15 0)
+      (effects (font (size 1.27 1.27)) hide)
+    )
+    (pin "1")
+    (pin "2")
+  )
   (symbol (lib_id "power:GNDD") (at 54.61 151.13 0) (unit 1)
     (in_bom yes) (on_board yes)
@@
     )
     (pin "1")
+  )
+  (symbol (lib_id "Device:R") (at 34.29 176.53 180) (unit 1)
+    (in_bom yes) (on_board yes)
+    (property "Reference" "R10" (id 0) (at 32.258 176.53 90))
+    (property "Value" "1k" (id 1) (at 36.83 176.53 90)
+      (effects (font (size 0.9906 0.9906)))
+    )
+    (property "Footprint" "Resistor_SMD:R_0603_1608Metric" (id 2) (at 36.068 176.53 90)
+      (effects (font (size 1.27 1.27)) hide)
+    )
+    (property "Datasheet" "" (id 3) (at 34.29 176.53 0)
+      (effects (font (size 1.27 1.27)) hide)
+    )
+    (pin "1")
+    (pin "2")
   )
   (symbol (lib_id "power:GNDD") (at 215.9 133.35 270) (unit 1)
@@
       (reference "#PWR024") (unit 1) (value "GNDD") (footprint "")
     )
+    (path "/6fd1cdf0-93d8-4be6-9ca8-a2d38a9f254a"
+      (reference "#PWR025") (unit 1) (value "GNDD") (footprint "")
+    )
     (path "/43d362e1-9459-4348-ab14-3501a2b74d02"
       (reference "#PWR026") (unit 1) (value "+5V") (footprint "")
@@
       (reference "C16") (unit 1) (value "330uF") (footprint "Capacitor_THT:CP_Radial_D10.0mm_P5.00mm")
     )
+    (path "/bf5ca043-be15-43ef-8cf4-c32cebb8dd56"
+      (reference "D1") (unit 1) (value "LED") (footprint "LED_SMD:LED_0603_1608Metric")
+    )
     (path "/eef9e806-a9b6-470d-9320-a07658a8b38f"
       (reference "D3") (unit 1) (value "S3JB") (footprint "Diode_SMD:D_SMB")
@@
     )
     (path "/5cc0177f-8bfd-4b5a-a860-188ac45a52ed"
-      (reference "Q1") (unit 1) (value "SI2306") (footprint "Package_TO_SOT_SMD:SOT-23")
+      (reference "Q1") (unit 1) (value "BSS138A") (footprint "Package_TO_SOT_SMD:SOT-23")
     )
     (path "/b46367c1-fa68-41db-b033-3080d7ab8ba9"
-      (reference "Q2") (unit 1) (value "Si2306") (footprint "Package_TO_SOT_SMD:SOT-23")
+      (reference "Q2") (unit 1) (value "BSS138A") (footprint "Package_TO_SOT_SMD:SOT-23")
     )
     (path "/1bcb394c-ff98-4a88-8c10-7a97fe99f772"
@@
       (reference "R9") (unit 1) (value "47k") (footprint "Resistor_SMD:R_0603_1608Metric")
     )
+    (path "/c8c086a8-4edc-4fcd-b56d-d6da757e451e"
+      (reference "R10") (unit 1) (value "1k") (footprint "Resistor_SMD:R_0603_1608Metric")
+    )
     (path "/00000000-0000-0000-0000-0000606cbb13"
